Commit message: added box urdf, fixed urdf errors

File: scout_description/urdf/example.urdf.xacro (robot description, xacro)
@@ -1,8 +1,4 @@
 <?xml version="1.0"?>
 <robot xmlns:xacro="http://www.ros.org/wiki/xacro" name="example">
-  <xacro:arg name="gpu" default="false"/>
-  <xacro:property name="gpu" value="$(arg gpu)" />
-  <xacro:arg name="organize_cloud" default="false"/>
-  <xacro:property name="organize_cloud" value="$(arg organize_cloud)" />
   <!-- Base Footprint -->
   <link name="base_footprint" />
@@ -36,4 +32,8 @@
     <origin xyz="0 0 0.4" rpy="0 0 0" />
   </xacro:VLP-16>
+  <xacro:include filename="$(find velodyne_description)/urdf/box_agile.xacro"/>
+  <xacro:box_agile>
+    <origin xyz="0 0 0.245" rpy="0 0 0" />
+  </xacro:box_agile>
   <xacro:include filename="$(find velodyne_description)/urdf/HDL-32E.urdf.xacro"/>
   <xacro:HDL-32E parent="base_link" name="velodyne2" topic="/velodyne_points2" organize_cloud="${organize_cloud}" hz="10" samples="220" gpu="${gpu}">

File: scout_description/urdf/mini.xacro (robot description, xacro)
@@ -8,4 +8,5 @@
     <xacro:include filename="$(find scout_description)/urdf/scout_mini_wheel_3.xacro" />
     <xacro:include filename="$(find scout_description)/urdf/scout_mini_wheel_4.xacro" />
+    <xacro:include filename="$(find scout_description)/urdf/box_agile.xacro"/>
     <!-- Variables -->
     <xacro:property name="M_PI" value="3.14159"/>
@@ -66,4 +67,7 @@
         <child link="base_link"/>
     </joint> -->
+    <!-- Agile Box initialization -->
+    <xacro:box_agile>
+    </xacro:box_agile>
     <!-- Scout wheel macros -->
     <!-- wheel labeled from 0 to 3, conter-clockwise, starting from front right wheel -->
@@ -105,5 +109,5 @@
   <xacro:include filename="$(find velodyne_description)/urdf/VLP-16.urdf.xacro"/>
   <xacro:VLP-16 parent="base_link" name="velodyne" topic="/velodyne_points" organize_cloud="${organize_cloud}" hz="10" samples="440" gpu="${gpu}">
-    <origin xyz="0 0 0.2" rpy="0 0 0" />
+    <origin xyz="0 0 0.1655" rpy="0 0 -${M_PI}" />
   </xacro:VLP-16>
   <!--<xacro:property name="M_PI" value="3.1415926535897931" />
