Commit message: Simplify wheels models

File: scout_description/urdf/scout_mini_wheel_1.xacro (robot description, xacro)
@@ -48,6 +48,9 @@
                 <origin xyz="0 0 0" rpy="0 0 0" />
                 <geometry>
-                    <mesh filename="package://scout_description/meshes/wheel.dae" />
+                    <mesh filename="package://scout_description/meshes/wheel_simple_big.stl" scale="0.001 0.001 0.001" />
                 </geometry>
+                <material name="black">
+                  <color rgba="0 0 0 1"/>
+                </material>
             </visual>
             <collision>
@@ -57,6 +60,9 @@
               <geometry>
                 <mesh
-                  filename="package://scout_description/meshes/wheel.dae" />
+                  filename="package://scout_description/meshes/wheel_simple_big.stl" scale="0.001 0.001 0.001" />
               </geometry>
+              <material name="black">
+                <color rgba="0 0 0 1"/>
+              </material>
             </collision>
         </link>

File: scout_description/urdf/scout_mini_wheel_2.xacro (robot description, xacro)
@@ -48,6 +48,9 @@
                 <origin xyz="0 0 0" rpy="0 0 0" />
                 <geometry>
-                    <mesh filename="package://scout_description/meshes/wheel.dae" />
+                    <mesh filename="package://scout_description/meshes/wheel_simple_big.stl" scale="0.001 0.001 0.001" />
                 </geometry>
+                <material name="black">
+                  <color rgba="0 0 0 1"/>
+                </material>
             </visual>
             <collision>
@@ -57,6 +60,9 @@
               <geometry>
                 <mesh
-                  filename="package://scout_description/meshes/wheel.dae" />
+                  filename="package://scout_description/meshes/wheel_simple_big.stl" scale="0.001 0.001 0.001" />
               </geometry>
+              <material name="black">
+                  <color rgba="0 0 0 1"/>
+                </material>
             </collision>
         </link>

File: scout_description/urdf/scout_mini_wheel_3.xacro (robot description, xacro)
@@ -48,6 +48,9 @@
                 <origin xyz="0 0 0" rpy="0 0 0" />
                 <geometry>
-                    <mesh filename="package://scout_description/meshes/wheel.dae" />
+                    <mesh filename="package://scout_description/meshes/wheel_simple_big.stl" scale="0.001 0.001 0.001" />
                 </geometry>
+                <material name="black">
+                  <color rgba="0 0 0 1"/>
+                </material>
             </visual>
             <collision>
@@ -57,6 +60,9 @@
               <geometry>
                 <mesh
-                  filename="package://scout_description/meshes/wheel.dae" />
+                  filename="package://scout_description/meshes/wheel_simple_big.stl" scale="0.001 0.001 0.001" />
               </geometry>
+              <material name="black">
+                  <color rgba="0 0 0 1"/>
+                </material>
             </collision>
         </link>

File: scout_description/urdf/scout_mini_wheel_4.xacro (robot description, xacro)
@@ -48,6 +48,9 @@
             <origin xyz="0 0 0" rpy="0 0 0" />
             <geometry>
-                <mesh filename="package://scout_description/meshes/wheel.dae" />
+                <mesh filename="package://scout_description/meshes/wheel_simple_big.stl" scale="0.001 0.001 0.001" />
             </geometry>
+            <material name="black">
+                  <color rgba="0 0 0 1"/>
+                </material>
         </visual>
             <collision>
@@ -57,6 +60,9 @@
               <geometry>
                 <mesh
-                  filename="package://scout_description/meshes/wheel.dae" />
+                  filename="package://scout_description/meshes/wheel_simple_big.stl" scale="0.001 0.001 0.001" />
               </geometry>
+              <material name="black">
+                  <color rgba="0 0 0 1"/>
+                </material>
             </collision>
         </link>

Commit message: Fixed wheels position

File: scout_description/urdf/scout_mini_wheel_1.xacro (robot description, xacro)
@@ -48,5 +48,5 @@
                 <origin xyz="0 0 0" rpy="0 0 0" />
                 <geometry>
-                    <mesh filename="package://scout_description/meshes/wheel_simple_big.stl" scale="0.001 0.001 0.001" />
+                    <mesh filename="package://scout_description/meshes/wheel_simple_short.stl" scale="0.001 0.001 0.001" />
                 </geometry>
                 <material name="black">
@@ -60,5 +60,5 @@
               <geometry>
                 <mesh
-                  filename="package://scout_description/meshes/wheel_simple_big.stl" scale="0.001 0.001 0.001" />
+                  filename="package://scout_description/meshes/wheel_simple_short.stl" scale="0.001 0.001 0.001" />
               </geometry>
               <material name="black">

File: scout_description/urdf/scout_mini_wheel_2.xacro (robot description, xacro)
@@ -48,5 +48,5 @@
                 <origin xyz="0 0 0" rpy="0 0 0" />
                 <geometry>
-                    <mesh filename="package://scout_description/meshes/wheel_simple_big.stl" scale="0.001 0.001 0.001" />
+                    <mesh filename="package://scout_description/meshes/wheel_simple_short.stl" scale="0.001 0.001 0.001" />
                 </geometry>
                 <material name="black">
@@ -60,5 +60,5 @@
               <geometry>
                 <mesh
-                  filename="package://scout_description/meshes/wheel_simple_big.stl" scale="0.001 0.001 0.001" />
+                  filename="package://scout_description/meshes/wheel_simple_short.stl" scale="0.001 0.001 0.001" />
               </geometry>
               <material name="black">

File: scout_description/urdf/scout_mini_wheel_3.xacro (robot description, xacro)
@@ -48,5 +48,5 @@
                 <origin xyz="0 0 0" rpy="0 0 0" />
                 <geometry>
-                    <mesh filename="package://scout_description/meshes/wheel_simple_big.stl" scale="0.001 0.001 0.001" />
+                    <mesh filename="package://scout_description/meshes/wheel_simple_short.stl" scale="0.001 0.001 0.001" />
                 </geometry>
                 <material name="black">
@@ -60,5 +60,5 @@
               <geometry>
                 <mesh
-                  filename="package://scout_description/meshes/wheel_simple_big.stl" scale="0.001 0.001 0.001" />
+                  filename="package://scout_description/meshes/wheel_simple_short.stl" scale="0.001 0.001 0.001" />
               </geometry>
               <material name="black">

File: scout_description/urdf/scout_mini_wheel_4.xacro (robot description, xacro)
@@ -48,5 +48,5 @@
             <origin xyz="0 0 0" rpy="0 0 0" />
             <geometry>
-                <mesh filename="package://scout_description/meshes/wheel_simple_big.stl" scale="0.001 0.001 0.001" />
+                <mesh filename="package://scout_description/meshes/wheel_simple_short.stl" scale="0.001 0.001 0.001" />
             </geometry>
             <material name="black">
@@ -60,5 +60,5 @@
               <geometry>
                 <mesh
-                  filename="package://scout_description/meshes/wheel_simple_big.stl" scale="0.001 0.001 0.001" />
+                  filename="package://scout_description/meshes/wheel_simple_short.stl" scale="0.001 0.001 0.001" />
               </geometry>
               <material name="black">
