Commit message: fix: solved an orientation problem

File: scout_description/urdf/mini.xacro (robot description, xacro)
@@ -109,5 +109,5 @@
   <xacro:include filename="$(find velodyne_description)/urdf/VLP-16.urdf.xacro"/>
   <xacro:VLP-16 parent="base_link" name="velodyne" topic="/velodyne_points" organize_cloud="${organize_cloud}" hz="10" samples="440" gpu="${gpu}">
-    <origin xyz="0 0 0.1655" rpy="0 0 -${M_PI}" />
+    <origin xyz="0 0 0.1655" rpy="0 0 0" />
   </xacro:VLP-16>
   <!--<xacro:property name="M_PI" value="3.1415926535897931" />

Commit message: Update robot model

File: scout_description/urdf/mini.xacro (robot description, xacro)
@@ -28,7 +28,7 @@
             <origin
                     xyz="0 0 0.0"
-                    rpy="1.57 0 -1.57" />
+                    rpy="0 0 -1.57" />
             <geometry>
-                <mesh filename="package://scout_description/meshes/scout_mini_base_link2.dae" />
+                <mesh filename="package://scout_description/meshes/scout_simple.stl" scale="0.001 0.001 0.001" />
             </geometry>
         </visual>
@@ -36,8 +36,8 @@
             <origin
                     xyz="0 0 0"
-                    rpy="1.57 0 -1.57" />
+                    rpy="0 0 -1.57" />
           <geometry>
             <mesh
-              filename="package://scout_description/meshes/scout_mini_base_link2.dae" />
+              filename="package://scout_description/meshes/scout_simple.stl" scale="0.001 0.001 0.001" />
           </geometry>
         </collision>

Commit message: Added IMU sensor

File: scout_description/urdf/mini.xacro (robot description, xacro)
@@ -251,3 +251,52 @@
       </xacro:unless>
     </gazebo>-->
+<!-- IMU -->
+<link name="imu_link">
+  <inertial>
+    <mass value="0.001"/>
+    <origin rpy="0 0 0" xyz="0 0 0"/>
+    <inertia ixx="0.0001" ixy="0" ixz="0" iyy="0.0001" iyz="0" izz="0.0001"/>
+  </inertial>
+  <visual>
+    <origin rpy="0 0 0" xyz="0 0 0"/>
+    <geometry>
+      <box size="0.1 0.1 0.1"/>
+    </geometry>
+  </visual>
+  <collision>
+    <origin rpy="0 0 0" xyz="0 0 0"/>
+    <geometry>
+      <box size="0.1 0.1 0.1"/>
+    </geometry>
+  </collision>
+</link>
+<!-- IMU Joint -->
+  <joint name="imu_joint" type="fixed">
+    <axis xyz="1 0 0"/> <!-- 0 1 0 -->
+    <origin xyz="0 0 0.28"/>
+    <parent link="base_link"/>
+    <child link="imu_link"/>
+  </joint>
+    <gazebo>
+    <!-- <plugin name="imu_plugin" filename="libgazebo_ros_imu.so">
+      <alwaysOn>true</alwaysOn>
+      <bodyName>base_link</bodyName>
+      <topicName>imu</topicName>
+      <serviceName>imu_service</serviceName>
+      <gaussianNoise>0.0</gaussianNoise>
+      <updateRate>100.0</updateRate>
+    </plugin> -->
+    <plugin name="imu_controller" filename="libhector_gazebo_ros_imu.so">
+      <robotNamespace>/</robotNamespace>
+      <updateRate>50.0</updateRate>
+      <bodyName>imu_link</bodyName>
+      <topicName>imu/data</topicName>
+      <accelDrift>0.005 0.005 0.005</accelDrift>
+      <accelGaussianNoise>0.005 0.005 0.005</accelGaussianNoise>
+      <rateDrift>0.005 0.005 0.005 </rateDrift>
+      <rateGaussianNoise>0.005 0.005 0.005 </rateGaussianNoise>
+      <headingDrift>0.005</headingDrift>
+      <headingGaussianNoise>0.005</headingGaussianNoise>
+    </plugin>
+    </gazebo>
 </robot>

Commit message: Lowered IMU joint

File: scout_description/urdf/mini.xacro (robot description, xacro)
@@ -274,5 +274,5 @@
   <joint name="imu_joint" type="fixed">
     <axis xyz="1 0 0"/> <!-- 0 1 0 -->
-    <origin xyz="0 0 0.28"/>
+    <origin xyz="0 0 0.1"/>
     <parent link="base_link"/>
     <child link="imu_link"/>
